File: LoRAK-v.2.kicad_pcb (KiCad board)
At the start: 2 copper layers, 90 x 90 mm, 7 parts, among them J1 UART, J2 I2C

Commit message: Add files via upload
Parts:
- added D1: LED, LED_SMD:LED_0402_1005Metric, F.Cu at (67.0, 93.3)
- added R2: R, Resistor_SMD:R_0603_1608Metric, F.Cu at (86.0, 113.7)
- added R3: R, Resistor_SMD:R_0603_1608Metric, F.Cu at (67.0, 97.3)
- added SW1: ~, 00_lib:PTS526, F.Cu at (87.7, 106.7)
- added SW3: ~, 00_lib:PTS526, F.Cu at (87.7, 97.0)
- J1: footprint Connector:FanPinHeader_1x04_P2.54mm_Vertical -> Connector_PinHeader_2.54mm:PinHeader_1x04_P2.54mm_Vertical
- J2: footprint Connector:NS-Tech_Grove_1x04_P2mm_Vertical -> 00_lib:Grove_2.0
- moved J2 12.9 mm to (95.0, 110.8)
- moved J1 7.82 mm to (73.2, 88.8), turned to 90 degrees
- moved C2 2.14 mm to (81.6, 96.0), turned to 90 degrees
- moved RAK3172(H)1 1.22 mm to (70.5, 109.3)
- moved U1 0.85 mm to (76.9, 97.5)
- moved C1 0.45 mm to (76.6, 93.4), turned to 0 degrees
Connections:
- RAK3172(H)1 pad 1: unconnected-(RAK3172(H)1-UART2_RX-Pad1) -> /RX
- RAK3172(H)1 pad 2: unconnected-(RAK3172(H)1-UART2_TX-Pad2) -> /TX
- RAK3172(H)1 pad 21: unconnected-(RAK3172(H)1-BOOT-Pad21) -> Net-(RAK3172(H)1-BOOT)
- RAK3172(H)1 pad 22: unconnected-(RAK3172(H)1-RST-Pad22) -> Net-(RAK3172(H)1-RST)
- RAK3172(H)1 pad 23: GND -> unconnected-(RAK3172(H)1-GND-Pad23)
- RAK3172(H)1 pad 32: unconnected-(RAK3172(H)1-ADC1-Pad32) -> Net-(RAK3172(H)1-ADC1)
- RAK3172(H)1 pad 4: /RX -> unconnected-(RAK3172(H)1-UART1_TX-Pad4)
- RAK3172(H)1 pad 5: /TX -> unconnected-(RAK3172(H)1-UART1_RX-Pad5)
Routing:
- net GND: track 32.9 -> 68.0 mm, vias 8 -> 6
- net Net-(RAK3172(H)1-RST): track 0.00 -> 32.4 mm
- net +3.3V: track 20.9 -> 47.4 mm
- net /RX: track 12.9 -> 32.2 mm
- net /TX: track 14.7 -> 30.6 mm
- net Net-(RAK3172(H)1-BOOT): track 0.00 -> 12.4 mm
- net /S1: track 24.5 -> 34.9 mm
- net /S2: track 30.5 -> 38.7 mm
- net Net-(RAK3172(H)1-ADC1): track 0.00 -> 3.54 mm
- net Net-(D1-A): track 0.00 -> 2.72 mm
- net /VIN: track 13.3 -> 10.7 mm
