File: LoRAK-v.2.kicad_sch (KiCad schematic)
At the start: 7 parts, among them J1 UART, J2 I2C

Commit message: Add files via upload
Parts:
- added D1: LED, LED_SMD:LED_0402_1005Metric, symbol Device:LED
- added R2, R3: R, Resistor_SMD:R_0603_1608Metric, symbol Device:R
- added SW1, SW3: ~, 00_lib:PTS526, symbol 00_Lib:PTS526
- J1: footprint Connector:FanPinHeader_1x04_P2.54mm_Vertical -> Connector_PinHeader_2.54mm:PinHeader_1x04_P2.54mm_Vertical
- J2: footprint Connector:NS-Tech_Grove_1x04_P2mm_Vertical -> 00_lib:Grove_2.0
Connections:
- net +3.3V: now also SW1.3, SW1.4
- net GND: now also D1.1 (K), R2.2, SW3.3, SW3.4; no longer RAK3172(H)1.23 (GND)
- net RX: now also RAK3172(H)1.1 (UART2_RX); no longer RAK3172(H)1.4 (UART1_TX)
- net TX: now also RAK3172(H)1.2 (UART2_TX); no longer RAK3172(H)1.5 (UART1_RX)
- net at RAK3172(H)1.21 (BOOT): now also R2.1, SW1.1, SW1.2
- net at RAK3172(H)1.22 (RST): now also SW3.1, SW3.2
- net at RAK3172(H)1.32 (ADC1): now also R3.2
- new net: D1.2 (A), R3.1
Other:
- moved on the sheet: J2
