File: CAD/Circuits-on-GNDplane/LoRAK-v.2.kicad_pcb (KiCad board)
At the start: 2 copper layers, 90 x 90 mm, 12 parts, among them J1 UART, J2 I2C

Commit message: update21Feb2024
Parts:
- renumbered J1 to UART
Other:
- board text added: "BOOT"
- board text added: "GND"
- board text added: "LoRAK v2.0"
- board text added: "Nov. 2023 CP 2xIFA BranchLine Coupler LEAT - F.P."
- board text added: "RESET"
- board text added: "Rx"
- board text added: "S1"
- board text added: "S2"
- board text added: "Tx"
- board text added: "Vin"
Changed lines of the file:
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@@
   (setup
     (pad_to_mask_clearance 0)
+    (aux_axis_origin 40.1 136.85)
+    (grid_origin 40.1 136.85)
     (pcbplotparams
       (layerselection 0x00010f0_ffffffff)
@@
     (property "ki_keywords" "connector")
     (attr through_hole)
-    (fp_text reference "J1" (at 0 -2.33 90) (layer "F.SilkS")
+    (fp_text reference "UART" (at 0 -2.33 90) (layer "F.SilkS")
         (effects (font (size 1 1) (thickness 0.15)))
     )
@@
   (gr_rect (start 40.1 46.85) (end 130.1 136.85)
     (stroke (width 0.1) (type default)) (fill none) (layer "Edge.Cuts"))
+  (gr_text "GND" (at 99.925 107.75) (layer "F.SilkS")
+    (effects (font (size 1 1) (thickness 0.15)))
+  )
+  (gr_text "Tx\n" (at 78.3 86.05) (layer "F.SilkS")
+    (effects (font (size 1 1) (thickness 0.15)))
+  )
+  (gr_text "GND" (at 73.05 86) (layer "F.SilkS")
+    (effects (font (size 1 1) (thickness 0.15)))
+  )
+  (gr_text "RESET\n" (at 92.5 97.175 270) (layer "F.SilkS")
+    (effects (font (size 1 1) (thickness 0.15)))
+  )
+  (gr_text "Vin\n" (at 75.9 86) (layer "F.SilkS")
+    (effects (font (size 1 1) (thickness 0.15)))
+  )
+  (gr_text "S1\n" (at 99.45 113.8) (layer "F.SilkS")
+    (effects (font (size 1 1) (thickness 0.15)))
+  )
+  (gr_text "S2" (at 99.5 111.8) (layer "F.SilkS")
+    (effects (font (size 1 1) (thickness 0.15)))
+  )
+  (gr_text "Rx" (at 80.825 86.1) (layer "F.SilkS")
+    (effects (font (size 1 1) (thickness 0.15)))
+  )
+  (gr_text "BOOT\n" (at 82.975 106.675 90) (layer "F.SilkS")
+    (effects (font (size 1 1) (thickness 0.15)))
+  )
+  (gr_text "Nov. 2023\nCP 2xIFA BranchLine Coupler\nLEAT - F.P." (at 41.1 135.825) (layer "F.SilkS")
+    (effects (font (size 0.7 0.7) (thickness 0.15)) (justify left bottom))
+  )
+  (gr_text "Vin\n" (at 99.6 109.8) (layer "F.SilkS")
+    (effects (font (size 1 1) (thickness 0.15)))
+  )
+  (gr_text "LoRAK v2.0" (at 41.1 132.05) (layer "F.SilkS")
+    (effects (font (size 0.8 0.8) (thickness 0.2) bold) (justify left bottom))
+  )
   (segment (start 63.327382 78.577382) (end 63.427382 78.577382) (width 0) (layer "F.Cu") (net 0))
   (segment (start 76.5025 98.1025) (end 76.6 98.005) (width 0.25) (layer "F.Cu") (net 1))
